File: release/v1.0-180804/controller.brd (EAGLE design)
At the start: 100 x 100 mm, 70 parts, among them J1 X, J10 FEED_HOLD, J11 PROBE, J12 ERROR, J13 HOLDING, J14 GND, J15 MOTOR_CURRENT, J16 SD_READER, J17 WHEEL, J19 Z_DISPLAY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

Commit message: added more documentation
Routing:
- net RADIO_RX: track 26.8 -> 28.0 mm
- net RADIO_TX: track 21.4 -> 22.4 mm
Changed lines of the file:
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@@
 <wire x1="46.355" y1="67.31" x2="53.848" y2="74.803" width="0.254" layer="16"/>
 <wire x1="53.848" y1="74.803" x2="56.261" y2="74.803" width="0.254" layer="16"/>
-<wire x1="56.261" y1="74.803" x2="56.388" y2="74.93" width="0.254" layer="16"/>
+<wire x1="56.261" y1="74.803" x2="56.388" y2="73.66" width="0.254" layer="16"/>
 </signal>
 <signal name="RADIO_RX">
@@
 <wire x1="51.7525" y1="64.77" x2="58.9915" y2="72.009" width="0.254" layer="16"/>
 <wire x1="58.9915" y1="72.009" x2="58.9915" y2="74.8665" width="0.254" layer="16"/>
-<wire x1="58.9915" y1="74.8665" x2="58.928" y2="74.93" width="0.254" layer="16"/>
+<wire x1="58.9915" y1="74.8665" x2="58.928" y2="73.66" width="0.254" layer="16"/>
 </signal>
 <signal name="FEED_OVERRIDE_OFF">
